Commit message: generated urdf based on new changes

File: yobo_model/yobotics_description/urdf/yobotics.urdf (robot description, URDF)
Before this commit: robot yobotics_description, 17 links, 16 joints
Links:
- added link imu_link, mass 0.001; collision box size=.001 .001 .001; visual box size=0.001 0.001 0.001
Joints:
- added joint imu_joint: type fixed, parent trunk, child imu_link, origin xyz=0 0 0 rpy=0 0 0
- joint FL_calf_joint: limit lower=-3.14159265359 upper=3.14159265359 effort=100 velocity=1.0 -> lower=-3.14159265359 upper=3.14159265359 effort=20 velocity=10.6
- joint FL_hip_joint: limit lower=-0.872664625997 upper=1.0471975512 effort=100 velocity=1.0 -> lower=-0.872664625997 upper=1.0471975512 effort=20 velocity=10.6
- joint FL_thigh_joint: limit lower=-0.523598775598 upper=3.92699081699 effort=100 velocity=1.0 -> lower=-0.523598775598 upper=3.92699081699 effort=20 velocity=10.6
- joint FR_calf_joint: limit lower=-3.14159265359 upper=3.14159265359 effort=100 velocity=1.0 -> lower=-3.14159265359 upper=3.14159265359 effort=20 velocity=10.6
- joint FR_hip_joint: limit lower=-1.0471975512 upper=0.872664625997 effort=100 velocity=1.0 -> lower=-1.0471975512 upper=0.872664625997 effort=20 velocity=10.6
- joint FR_thigh_joint: limit lower=-0.523598775598 upper=3.92699081699 effort=100 velocity=1.0 -> lower=-0.523598775598 upper=3.92699081699 effort=20 velocity=10.6
- joint RL_calf_joint: limit lower=-3.14159265359 upper=3.14159265359 effort=100 velocity=1.0 -> lower=-3.14159265359 upper=3.14159265359 effort=20 velocity=10.6
- joint RL_hip_joint: limit lower=-0.872664625997 upper=1.0471975512 effort=100 velocity=1.0 -> lower=-0.872664625997 upper=1.0471975512 effort=20 velocity=10.6
- joint RL_thigh_joint: limit lower=-0.523598775598 upper=3.92699081699 effort=100 velocity=1.0 -> lower=-0.523598775598 upper=3.92699081699 effort=20 velocity=10.6
- joint RR_calf_joint: limit lower=-3.14159265359 upper=3.14159265359 effort=100 velocity=1.0 -> lower=-3.14159265359 upper=3.14159265359 effort=20 velocity=10.6
- joint RR_hip_joint: limit lower=-1.0471975512 upper=0.872664625997 effort=100 velocity=1.0 -> lower=-1.0471975512 upper=0.872664625997 effort=20 velocity=10.6
- joint RR_thigh_joint: limit lower=-0.523598775598 upper=3.92699081699 effort=100 velocity=1.0 -> lower=-0.523598775598 upper=3.92699081699 effort=20 velocity=10.6

Commit message: working gazebo model

File: yobo_model/yobotics_description/urdf/yobotics.urdf (robot description, URDF)
Before this commit: robot yobotics_description, 18 links, 17 joints
Links:
- added link camera_depth_frame
- added link camera_depth_optical_frame
- added link camera_link, mass 0.200; collision mesh filename=package://hector_sensors_description/meshes/asus_camera/asu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; visual mesh filename=package://hector_sensors_description/meshes/asus_camera/asu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
- added link camera_rgb_frame
- added link camera_rgb_optical_frame
- added link hokuyo_frame, mass 0.270; collision box size=0.058 0.058 0.087; visual mesh filename=package://hector_sensors_description/meshes/hokuyo_utm30lx/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
- added link trunk_interia, mass 3.3; collision mesh filename=package://yobotics_description/meshes/trunk.STL scale=1 1 1; visual mesh filename=package://yobotics_description/meshes/trunk.STL scale=1 1 1
- link imu_link: geometry 
- link trunk: mass 3.3 -> None; geometry 
Joints:
- added joint camera_depth_joint: type fixed, parent camera_link, child camera_depth_frame, origin xyz=0.0 0.049 0.0 rpy=0 0 0
- added joint camera_depth_optical_joint: type fixed, parent camera_depth_frame, child camera_depth_optical_frame, origin xyz=0 0 0 rpy=-1.57079632679 0.0 -1.57079632679
- added joint camera_joint: type fixed, parent trunk, child camera_link, origin xyz=0.1 0.0 -0.06 rpy=0 0.261799612195482 0
- added joint camera_rgb_joint: type fixed, parent camera_link, child camera_rgb_frame, origin xyz=0.0 0.022 0.0 rpy=0 0 0
- added joint camera_rgb_optical_joint: type fixed, parent camera_rgb_frame, child camera_rgb_optical_frame, origin xyz=0 0 0 rpy=-1.57079632679 0.0 -1.57079632679
- added joint hokuyo_joint: type fixed, parent trunk, child hokuyo_frame, origin xyz=0.0 0.0 0.09375 rpy=0 0 0
- added joint trunk_to_trunk_inertia: type fixed, parent trunk, child trunk_interia, origin xyz=0 0 0 rpy=0 0 0
- joint FL_foot_fixed: origin xyz=0 0.0096 -0.21039 rpy=0 0 0 -> xyz=0 0 -0.23039 rpy=0 0 0
- joint FR_foot_fixed: origin xyz=0 0.0096 -0.21039 rpy=0 0 0 -> xyz=0 0 -0.23039 rpy=0 0 0
- joint RL_foot_fixed: origin xyz=0 0.0096 -0.21039 rpy=0 0 0 -> xyz=0 0 -0.23039 rpy=0 0 0
- joint RR_foot_fixed: origin xyz=0 0.0096 -0.21039 rpy=0 0 0 -> xyz=0 0 -0.23039 rpy=0 0 0
- joint imu_joint: origin xyz=0 0 0 rpy=0 0 0 -> (none)

File: yobo_model/yobotics_description/xacro/const.xacro (robot description, xacro)
@@ -16,5 +16,5 @@
     <xacro:property name="calf_length" value="0.016"/>
     <xacro:property name="calf_width" value="0.016"/>
-    <xacro:property name="calf_height" value="0.21039"/>
+    <xacro:property name="calf_height" value="0.23039"/>
     <xacro:property name="foot_radius" value="0.0265"/>
     <xacro:property name="stick_radius" value="0.01"/>

File: yobo_model/yobotics_description/xacro/gazebo.xacro (robot description, xacro)
@@ -25,7 +25,7 @@
         </plugin>
     </gazebo>
-    <gazebo reference="imu_link">
+    <!-- <gazebo reference="imu_link">
         <gravity>true</gravity>
-        <sensor name="imu_sensor" type="imu">
+        <sensor name="_sensor" type="imu">
             <always_on>true</always_on>
             <update_rate>1000</update_rate>
@@ -43,5 +43,5 @@
             <pose>0 0 0 0 0 0</pose>
         </sensor>
-    </gazebo>
+    </gazebo> -->
     <gazebo>
     <plugin filename="libgazebo_ros_p3d.so" name="p3d_base_controller">

File: yobo_model/yobotics_description/xacro/leg.xacro (robot description, xacro)
@@ -141,5 +141,5 @@
 <!-- //////////////////////foot//////////////////// -->
         <joint name="${name}_foot_fixed" type="fixed">
-            <origin rpy="0 0 0" xyz="0 ${foot_offset_y} ${-(calf_height)}"/>
+            <origin rpy="0 0 0" xyz="0 0 ${-(calf_height)}"/>
             <parent link="${name}_calf"/>
             <child link="${name}_foot"/>
@@ -147,5 +147,5 @@
         <link name="${name}_foot">
             <visual>
-                <origin rpy="0 0 0" xyz="0 0 0"/>
+                <origin rpy="0 0 0" xyz="0 0.009 0.02"/>
                 <geometry>
                      <mesh filename="package://yobotics_description/meshes/foot.STL" scale="1 1 1"/>
@@ -154,5 +154,5 @@
             </visual>
             <collision>
-                <origin rpy="0 0 0" xyz="0 0 0"/>
+                <origin rpy="0 0 0" xyz="0 0.009 0.02"/>
                 <geometry>
                     <mesh filename="package://yobotics_description/meshes/foot.STL" scale="1 1 1"/>

File: yobo_model/yobotics_description/xacro/robot.xacro (robot description, xacro)
@@ -19,5 +19,6 @@
         <child link="trunk"/>
     </joint> -->
-    <link name="trunk">
+    <link name="trunk"/>
+    <link name="trunk_interia">
         <visual>
             <origin rpy="0 0 0" xyz="0 0 0"/>
@@ -28,5 +29,5 @@
         </visual>
         <collision>
-            <origin rpy="0 0 0" xyz="0 0 ${trunk_offset_z}"/>
+            <origin rpy="0 0 0" xyz="0 0 0"/>
             <geometry>
                <mesh filename="package://yobotics_description/meshes/trunk.STL" scale="1 1 1"/>
@@ -43,4 +44,10 @@
         </inertial>
     </link>
+   <joint name="trunk_to_trunk_inertia" type="fixed">
+        <origin rpy="0 0 0" xyz="0 0 0"/>
+        <parent link="trunk"/>
+        <child link="trunk_interia"/>
+    </joint>
+<!--
     <joint name="imu_joint" type="fixed">
         <parent link="trunk"/>
@@ -67,5 +74,5 @@
             </geometry>
         </collision>
-    </link>
+    </link> -->
     <xacro:leg name="RL" mirror="-1" mirror_dae="False" front_hind="1" front_hind_dae="True">
         <origin rpy="0 0 0" xyz="${leg_offset_x} ${-leg_offset_y} 0"/>
@@ -80,3 +87,4 @@
         <origin rpy="0 0 0" xyz="${-leg_offset_x} ${leg_offset_y} 0"/>
     </xacro:leg>
+    <xacro:include filename="$(find yobotics_description)/xacro/accessories.urdf.xacro" />
 </robot>

Commit message: fixed misaligned frames and changed to boxed collisions

File: yobo_model/yobotics_description/urdf/yobotics.urdf (robot description, URDF)
Before this commit: robot yobotics_description, 25 links, 24 joints
Links:
- link FL_calf: geometry collision box size=0.016 0.016 0.2; visual mesh filename=package://yobotics_description/meshes/calf.STL scale=1 1 1
- link FL_foot: geometry collision sphere radius=0.025; visual mesh filename=package://yobotics_description/meshes/foot.STL scale=1 1 1
- link FL_hip: geometry collision box size=0.09 0.08 0.093; visual mesh filename=package://yobotics_description/meshes/hip.STL scale=1 1 1
- link FL_thigh: geometry collision box size=0.043 0.034 0.22; visual mesh filename=package://yobotics_description/meshes/thigh.STL scale=1 1 1
- link FR_calf: geometry collision box size=0.016 0.016 0.2; visual mesh filename=package://yobotics_description/meshes/calf.STL scale=1 1 1
- link FR_foot: geometry collision sphere radius=0.025; visual mesh filename=package://yobotics_description/meshes/foot.STL scale=1 1 1
- link FR_hip: geometry collision box size=0.09 0.08 0.093; visual mesh filename=package://yobotics_description/meshes/hip.STL scale=1 1 1
- link FR_thigh: geometry collision box size=0.043 0.034 0.22; visual mesh filename=package://yobotics_description/meshes/thigh.STL scale=1 1 1
- link RL_calf: geometry collision box size=0.016 0.016 0.2; visual mesh filename=package://yobotics_description/meshes/calf.STL scale=1 1 1
- link RL_foot: geometry collision sphere radius=0.025; visual mesh filename=package://yobotics_description/meshes/foot.STL scale=1 1 1
- link RL_hip: geometry collision box size=0.09 0.08 0.093; visual mesh filename=package://yobotics_description/meshes/hip.STL scale=1 1 1
- link RL_thigh: geometry collision box size=0.043 0.034 0.22; visual mesh filename=package://yobotics_description/meshes/thigh.STL scale=1 1 1
- link RR_calf: geometry collision box size=0.016 0.016 0.2; visual mesh filename=package://yobotics_description/meshes/calf.STL scale=1 1 1
- link RR_foot: geometry collision sphere radius=0.025; visual mesh filename=package://yobotics_description/meshes/foot.STL scale=1 1 1
- link RR_hip: geometry collision box size=0.09 0.08 0.093; visual mesh filename=package://yobotics_description/meshes/hip.STL scale=1 1 1
- link RR_thigh: geometry collision box size=0.043 0.034 0.22; visual mesh filename=package://yobotics_description/meshes/thigh.STL scale=1 1 1
- link trunk_interia: geometry collision box size=0.3 0.2 0.093; visual mesh filename=package://yobotics_description/meshes/trunk.STL scale=1 1 1
Joints:
- joint FL_calf_joint: origin xyz=0 0.0106 -0.2115 rpy=0 0 0 -> xyz=0 0 -0.2115 rpy=0 0 0
- joint FR_calf_joint: origin xyz=0 0.0106 -0.2115 rpy=0 0 0 -> xyz=0 0 -0.2115 rpy=0 0 0
- joint RL_calf_joint: origin xyz=0 0.0106 -0.2115 rpy=0 0 0 -> xyz=0 0 -0.2115 rpy=0 0 0
- joint RR_calf_joint: origin xyz=0 0.0106 -0.2115 rpy=0 0 0 -> xyz=0 0 -0.2115 rpy=0 0 0
- joint hokuyo_joint: origin xyz=0.0 0.0 0.09375 rpy=0 0 0 -> xyz=0.0 0.0 0.093 rpy=0 0 0

File: yobo_model/yobotics_description/xacro/accessories.urdf.xacro (robot description, xacro)
@@ -11,5 +11,5 @@
         min_angle="130"
         max_angle="-130" >
-        <origin xyz="0.0 0.0 ${trunk_height / 2}" rpy="0 0 0"/>
+        <origin xyz="0.0 0.0 ${trunk_height}" rpy="0 0 0"/>
     </xacro:hokuyo_utm30lx>
     <gazebo reference="hokuyo_frame">

File: yobo_model/yobotics_description/xacro/const.xacro (robot description, xacro)
@@ -5,16 +5,16 @@
     <xacro:property name="stick_mass" value="0.00001"/>
     <!-- simplified collision value -->
-    <xacro:property name="trunk_length" value="0.5616"/>
-    <xacro:property name="trunk_width" value="0.172"/>
-    <xacro:property name="trunk_height" value="0.1875"/>
-    <xacro:property name="hip_length" value="0.08"/>
+    <xacro:property name="trunk_length" value="0.3"/>
+    <xacro:property name="trunk_width" value="0.20"/>
+    <xacro:property name="trunk_height" value="0.093"/>
+    <xacro:property name="hip_length" value="0.09"/>
     <xacro:property name="hip_width" value="0.08"/>
-    <xacro:property name="hip_height" value="0.08"/>
+    <xacro:property name="hip_height" value="0.093"/>
     <xacro:property name="thigh_length" value="0.043"/>
     <xacro:property name="thigh_width" value="0.034"/>
-    <xacro:property name="thigh_height" value="0.2115"/>
+    <xacro:property name="thigh_height" value="0.22"/>
     <xacro:property name="calf_length" value="0.016"/>
     <xacro:property name="calf_width" value="0.016"/>
-    <xacro:property name="calf_height" value="0.23039"/>
+    <xacro:property name="calf_height" value="0.20"/>
     <xacro:property name="foot_radius" value="0.0265"/>
     <xacro:property name="stick_radius" value="0.01"/>

File: yobo_model/yobotics_description/xacro/leg.xacro (robot description, xacro)
@@ -39,5 +39,5 @@
             <collision>
                 <!-- <origin rpy="${PI/2.0} 0 0" xyz="0 0 0"/> -->
-                <xacro:if value="${(mirror_dae == True) and (front_hind_dae == True)}">
+                <!-- <xacro:if value="${(mirror_dae == True) and (front_hind_dae == True)}">
                     <origin rpy="0 0 0" xyz="0 0 0"/>
                 </xacro:if>
@@ -50,7 +50,8 @@
                 <xacro:if value="${(mirror_dae == False) and (front_hind_dae == False)}">
                     <origin rpy="${PI} ${PI} 0" xyz="0 0 0"/>
-                </xacro:if>
+                </xacro:if> -->
                 <geometry>
-                    <mesh filename="package://yobotics_description/meshes/hip.STL" scale="1 1 1"/>
+                    <!-- <mesh filename="package://yobotics_description/meshes/hip.STL" scale="1 1 1"/> -->
+                    <box size="${hip_length} ${hip_width} ${hip_height}"/>
                 </geometry>
             </collision>
@@ -65,5 +66,5 @@
 <!-- //////////////////////thigh//////////////////// -->
         <joint name="${name}_thigh_joint" type="revolute">
-         <!-- <joint name="${name}_thigh_joint" type="continuous"> -->
+        <!-- <joint name="${name}_thigh_joint" type="continuous"> -->
             <origin rpy="0 0 0" xyz="0 ${-thigh_offset*mirror} 0"/>
             <parent link="${name}_hip"/>
@@ -87,12 +88,14 @@
             </visual>
             <collision>
-                 <xacro:if value="${mirror_dae == True}">
+                 <!-- <xacro:if value="${mirror_dae == True}">
                     <origin rpy="0 0 0" xyz="0 0 0"/>
                 </xacro:if>
                 <xacro:if value="${mirror_dae == False}">
                     <origin rpy="${PI} ${PI} 0" xyz="0 0 0"/>
-                </xacro:if>
+                </xacro:if> -->
+                <origin rpy="0 0 0" xyz="0 0 -${thigh_height / 2}"/>
                 <geometry>
-                    <mesh filename="package://yobotics_description/meshes/thigh.STL" scale="1 1 1"/>
+                    <box size="${thigh_length} ${thigh_width} ${thigh_height}"/>
+                    <!-- <mesh filename="package://yobotics_description/meshes/thigh.STL" scale="1 1 1"/> -->
                 </geometry>
                 <material name="white_blue"/>
@@ -109,5 +112,5 @@
         <joint name="${name}_calf_joint" type="revolute">
         <!-- <joint name="${name}_calf_joint" type="continuous"> -->
-            <origin rpy="0 0 0" xyz="0 ${calf_offset_y} ${-thigh_height}"/>
+            <origin rpy="0 0 0" xyz="0 0 -0.2115"/>
             <parent link="${name}_thigh"/>
             <child link="${name}_calf"/>
@@ -119,5 +122,5 @@
         <link name="${name}_calf">
             <visual>
-                <origin rpy="0 0 0" xyz="0.0 0.0 0.0" />
+                <origin rpy="0 0 0" xyz="0.0 0.009 0.0" />
                 <geometry>
                     <mesh filename="package://yobotics_description/meshes/calf.STL" scale="1 1 1"/>
@@ -126,7 +129,8 @@
             </visual>
             <collision>
-                <origin rpy="0 0 0" xyz="0.0 0.0 0.0" />
+                <origin rpy="0 0 0" xyz="0.0 0.0 -${calf_height / 2}" />
                 <geometry>
-                    <mesh filename="package://yobotics_description/meshes/calf.STL" scale="1 1 1"/>
+                    <box size="${calf_length} ${calf_width} ${calf_height}"/>
+                    <!-- <mesh filename="package://yobotics_description/meshes/calf.STL" scale="1 1 1"/> -->
                 </geometry>
             </collision>
@@ -141,5 +145,5 @@
 <!-- //////////////////////foot//////////////////// -->
         <joint name="${name}_foot_fixed" type="fixed">
-            <origin rpy="0 0 0" xyz="0 0 ${-(calf_height)}"/>
+            <origin rpy="0 0 0" xyz="0 0 -0.23039"/>
             <parent link="${name}_calf"/>
             <child link="${name}_foot"/>
@@ -147,5 +151,5 @@
         <link name="${name}_foot">
             <visual>
-                <origin rpy="0 0 0" xyz="0 0.009 0.02"/>
+                <origin rpy="0 0 0" xyz="0 0.018 0.02"/>
                 <geometry>
                      <mesh filename="package://yobotics_description/meshes/foot.STL" scale="1 1 1"/>
@@ -154,7 +158,8 @@
             </visual>
             <collision>
-                <origin rpy="0 0 0" xyz="0 0.009 0.02"/>
+                <origin rpy="0 0 0" xyz="0 0.0 0.025"/>
                 <geometry>
-                    <mesh filename="package://yobotics_description/meshes/foot.STL" scale="1 1 1"/>
+                    <!-- <mesh filename="package://yobotics_description/meshes/foot.STL" scale="1 1 1"/> -->
+                    <sphere radius="0.025"/>
                 </geometry>
             </collision>

File: yobo_model/yobotics_description/xacro/robot.xacro (robot description, xacro)
@@ -31,6 +31,6 @@
             <origin rpy="0 0 0" xyz="0 0 0"/>
             <geometry>
-               <mesh filename="package://yobotics_description/meshes/trunk.STL" scale="1 1 1"/>
-               <!-- <box size="${trunk_length} ${trunk_width} ${trunk_height}"/> -->
+               <!-- <mesh filename="package://yobotics_description/meshes/trunk.STL" scale="1 1 1"/> -->
+               <box size="${trunk_length} ${trunk_width} ${trunk_height}"/>
             </geometry>
         </collision>
